File: MD-AM2837/MD-AM2837.kicad_sch (KiCad schematic)
At the start: 13 parts, among them J1 XT60_Male_Horizontal, J2 XT60_Female_Horizontal, J3 Conn_01x03_Pin_signal

Commit message: タイトルと名前を記入した
Other:
- company: (none) -> 明治大学オートメーション研究部
- title: (none) -> モータードライバ基板（弱）
Changed lines of the file:
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@@
 	(generator_version "8.0")
 	(paper "A4")
+	(title_block
+		(title "モータードライバ基板（弱）")
+		(date "2024-09-30")
+		(rev "1")
+		(company "明治大学オートメーション研究部")
+		(comment 1 "次田英太")
+		(comment 2 "電気電子生命学科2年")
+	)
 	(junction
 		(at 102.87 95.25)
